File: door/door_board.sch (EAGLE design)
At the start: 40 parts, among them IC1 MCP1703CB, IC2 MCP601OT, IC3 AP1609SOP8, Q1 4.3A/20V/54mΩ, T2 BC847

Commit message: Updated board to version 1.1
Fixed VCC to nrf
Flipped HV enable high side mosfet
Corrected AP1609 footprint
Updated board text
Parts:
- RESET: value (none) -> MOMENTARY-SWITCH-SPST-PTH-6.0MM; device adafruit:SWITCH_PUSHBUTTONSOFTTOUCHSMD_SJ -> SparkFun-Switches:MOMENTARY-SWITCH-SPST-PTH-6.0MM
- renumbered U$2 to XTAL
Connections:
- net N$4 renamed RX
- net N$5 renamed TX
- net 3V3: now also U$1.VDD_NRF
- net GND: now also RESET.2; no longer RESET.P$2
- net NRST: now also RESET.1; no longer RESET.P$1
- net VIN: now also Q1.S; no longer Q1.D
- net VIN_CONT: now also Q1.D; no longer Q1.S
Other:
- moved on the sheet: Q1
Changed lines of the file:
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@@
 </classes>
 <parts>
-<part name="U$2" library="BLE" deviceset="QANXTAL" device=""/>
+<part name="XTAL" library="BLE" deviceset="QANXTAL" device=""/>
 <part name="C1" library="rcl" library_urn="urn:adsk.eagle:library:334" deviceset="C-EU" device="C0603" package3d_urn="urn:adsk.eagle:package:23616/2" value="12 pF"/>
 <part name="C2" library="rcl" library_urn="urn:adsk.eagle:library:334" deviceset="C-EU" device="C0603" package3d_urn="urn:adsk.eagle:package:23616/2" value="12 pF"/>
@@
 <part name="GND5" library="supply1" library_urn="urn:adsk.eagle:library:371" deviceset="GND" device=""/>
 <part name="PRGM" library="pinhead" library_urn="urn:adsk.eagle:library:325" deviceset="PINHD-1X5" device="" package3d_urn="urn:adsk.eagle:package:22469/2"/>
-<part name="RESET" library="adafruit" library_urn="urn:adsk.eagle:library:420" deviceset="SWITCH_PUSHBUTTON" device="SOFTTOUCHSMD_SJ" package3d_urn="urn:adsk.eagle:package:6240956/1"/>
+<part name="RESET" library="SparkFun-Switches" deviceset="MOMENTARY-SWITCH-SPST" device="-PTH-6.0MM"/>
 <part name="GND7" library="supply1" library_urn="urn:adsk.eagle:library:371" deviceset="GND" device=""/>
 <part name="LED1" library="adafruit" library_urn="urn:adsk.eagle:library:420" deviceset="LED" device="CHIP-LED0805" package3d_urn="urn:adsk.eagle:package:6240557/1" value="Red"/>
@@
 </plain>
 <instances>
-<instance part="U$2" gate="G$1" x="-20.32" y="-53.34" smashed="yes" rot="R270">
+<instance part="XTAL" gate="G$1" x="-20.32" y="-53.34" smashed="yes" rot="R270">
 <attribute name="NAME" x="-19.304" y="-55.88" size="1.778" layer="95" rot="R270"/>
 <attribute name="VALUE" x="-22.86" y="-55.88" size="1.778" layer="96" rot="R270"/>
@@
 <attribute name="VALUE" x="-284.48" y="-33.02" size="1.778" layer="96"/>
 </instance>
-<instance part="Q1" gate="G$1" x="-254" y="-25.4" smashed="yes">
-<attribute name="NAME" x="-248.92" y="-25.4" size="1.778" layer="95" font="vector"/>
-<attribute name="VALUE" x="-248.92" y="-27.94" size="1.778" layer="96" font="vector"/>
+<instance part="Q1" gate="G$1" x="-254" y="-25.4" smashed="yes" rot="MR180">
+<attribute name="NAME" x="-248.92" y="-25.4" size="1.778" layer="95" font="vector" rot="MR180"/>
+<attribute name="VALUE" x="-248.92" y="-22.86" size="1.778" layer="96" font="vector" rot="MR180"/>
 </instance>
 <instance part="R10" gate="G$1" x="-287.02" y="-38.1" smashed="yes">
@@
 <net name="N$1" class="0">
 <segment>
-<pinref part="U$2" gate="G$1" pin="1"/>
+<pinref part="XTAL" gate="G$1" pin="1"/>
 <wire x1="-2.54" y1="-50.8" x2="-20.32" y2="-50.8" width="0.1524" layer="91"/>
 <pinref part="C1" gate="G$1" pin="1"/>
@@
 <net name="N$2" class="0">
 <segment>
-<pinref part="U$2" gate="G$1" pin="2"/>
+<pinref part="XTAL" gate="G$1" pin="2"/>
 <wire x1="-5.08" y1="-55.88" x2="-20.32" y2="-55.88" width="0.1524" layer="91"/>
 <pinref part="C2" gate="G$1" pin="1"/>
@@
 </segment>
 <segment>
-<pinref part="RESET" gate="G$1" pin="P$2"/>
+<pinref part="RESET" gate="G$1" pin="2"/>
 <wire x1="99.06" y1="-63.5" x2="111.76" y2="-63.5" width="0.1524" layer="91"/>
 <wire x1="111.76" y1="-63.5" x2="111.76" y2="-68.58" width="0.1524" layer="91"/>
@@
 </segment>
 <segment>
-<pinref part="Q1" gate="G$1" pin="D"/>
-<wire x1="-251.46" y1="-20.32" x2="-251.46" y2="-5.08" width="0.1524" layer="91"/>
 <pinref part="R12" gate="G$1" pin="2"/>
 <wire x1="-251.46" y1="-5.08" x2="-271.78" y2="-5.08" width="0.1524" layer="91"/>
@@
 <junction x="-271.78" y="-5.08"/>
 <label x="-271.78" y="5.08" size="1.778" layer="95" rot="R90" xref="yes"/>
+<pinref part="Q1" gate="G$1" pin="S"/>
+<wire x1="-251.46" y1="-5.08" x2="-251.46" y2="-20.32" width="0.1524" layer="91"/>
 </segment>
 <segment>
@@
 <label x="93.98" y="-25.4" size="1.778" layer="95" rot="R180" xref="yes"/>
 </segment>
+<segment>
+<pinref part="U$1" gate="G$1" pin="VDD_NRF"/>
+<wire x1="-7.62" y1="-40.64" x2="-7.62" y2="-45.72" width="0.1524" layer="91"/>
+<wire x1="-7.62" y1="-45.72" x2="-12.7" y2="-45.72" width="0.1524" layer="91"/>
+<label x="-12.7" y="-45.72" size="1.778" layer="95" rot="R180"/>
+</segment>
 </net>
 <net name="ADFSGSDFH" class="0">
@@
 <pinref part="Q1" gate="G$1" pin="G"/>
 <wire x1="-271.78" y1="-27.94" x2="-271.78" y2="-22.86" width="0.1524" layer="91"/>
-<wire x1="-259.08" y1="-27.94" x2="-271.78" y2="-27.94" width="0.1524" layer="91"/>
+<wire x1="-259.08" y1="-22.86" x2="-271.78" y2="-27.94" width="0.1524" layer="91"/>
 <junction x="-271.78" y="-27.94"/>
 </segment>
@@
 <net name="VIN_CONT" class="0">
 <segment>
-<pinref part="Q1" gate="G$1" pin="S"/>
-<wire x1="-251.46" y1="-30.48" x2="-251.46" y2="-33.02" width="0.1524" layer="91"/>
 <wire x1="-251.46" y1="-33.02" x2="-246.38" y2="-33.02" width="0.1524" layer="91"/>
 <label x="-246.38" y="-33.02" size="1.778" layer="95" xref="yes"/>
+<pinref part="Q1" gate="G$1" pin="D"/>
+<wire x1="-251.46" y1="-30.48" x2="-251.46" y2="-33.02" width="0.1524" layer="91"/>
 </segment>
 <segment>
@@
 </segment>
 <segment>
-<pinref part="RESET" gate="G$1" pin="P$1"/>
+<pinref part="RESET" gate="G$1" pin="1"/>
 <wire x1="88.9" y1="-63.5" x2="81.28" y2="-63.5" width="0.1524" layer="91"/>
 <label x="81.28" y="-63.5" size="1.778" layer="95" rot="R180" xref="yes"/>
@@
 </segment>
 </net>
-<net name="N$4" class="0">
+<net name="RX" class="0">
 <segment>
 <pinref part="U$1" gate="G$1" pin="SIO_08/UART_RX"/>
@@
 <wire x1="15.24" y1="-40.64" x2="15.24" y2="-71.12" width="0.1524" layer="91"/>
 <wire x1="15.24" y1="-71.12" x2="43.18" y2="-71.12" width="0.1524" layer="91"/>
-</segment>
-</net>
-<net name="N$5" class="0">
+<label x="15.24" y="-53.34" size="1.778" layer="95"/>
+</segment>
+</net>
+<net name="TX" class="0">
 <segment>
 <pinref part="UART" gate="A" pin="1"/>
@@
 <wire x1="43.18" y1="-68.58" x2="10.16" y2="-68.58" width="0.1524" layer="91"/>
 <wire x1="10.16" y1="-68.58" x2="10.16" y2="-40.64" width="0.1524" layer="91"/>
-</segment>
-</net>
+<label x="5.08" y="-55.88" size="1.778" layer="95"/>
+</segment>
+</net>
